File: Hardware/Dosimeter/Dosimeter.sch (KiCad schematic (older format))
At the start: 43 parts, among them J1 USB_B_Mini, J2 Vin +12, J3 Conn_01x01_Female, J4 Conn_01x01_Female, J5 Conn_01x02_Male, J6 Conn_01x02_Male, J7 Conn_01x01_Female, Q1 BC846, SW1 SW_Push, SW2 SW_Push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

Commit message: complete HW, add Software
Parts:
- added BT1: Battery, MK_Footprints:BatteryHolder_Keystone_2477_4xAA, symbol Device:Battery
- added J8: Conn_01x04_Male, Connector_PinHeader_2.54mm:PinHeader_1x04_P2.54mm_Vertical, symbol Connector:Conn_01x04_Male
- C10: value 47p -> 100p; footprint Capacitor_THT:C_Disc_D8.0mm_W5.0mm_P10.00mm -> Capacitor_THT:C_Axial_L3.8mm_D2.6mm_P12.50mm_Horizontal
Connections:
- net +3V3: now also J8.1 (Pin_1)
- net +6V: now also RV1.3, BT1.1 (+)
- net GND: now also BT1.2 (-), J8.4 (Pin_4)
- net at R10.1, U5.1: no longer RV1.3
- net SWDIO: now reaches U2.23 (PA13)
- net SWDIO: now also J8.3 (Pin_3)
- net SWCLK: now reaches U2.24 (PA14)
- net SWCLK: now also J8.2 (Pin_2)
- no-connect marks 9 -> 7
Other:
- moved on the sheet: RV1
Changed lines of the file:
@@
 P 4050 2250
 F 0 "C10" V 3798 2250 50  0000 C CNN
-F 1 "47p" V 3889 2250 50  0000 C CNN
-F 2 "Capacitor_THT:C_Disc_D8.0mm_W5.0mm_P10.00mm" H 4088 2100 50  0001 C CNN
+F 1 "100p" V 3889 2250 50  0000 C CNN
+F 2 "Capacitor_THT:C_Axial_L3.8mm_D2.6mm_P12.50mm_Horizontal" H 4088 2100 50  0001 C CNN
 F 3 "~" H 4050 2250 50  0001 C CNN
 	1    4050 2250
@@
 Wire Wire Line
 	5550 2950 5500 2950
-Wire Wire Line
-	6150 2850 6250 2850
 $Comp
 L Device:R_POT RV1
 U 1 1 5F48F410
-P 6250 3300
-F 0 "RV1" H 6181 3346 50  0000 R CNN
-F 1 "R_POT" H 6181 3255 50  0000 R CNN
-F 2 "Potentiometer_THT:Potentiometer_Vishay_T73YP_Vertical" H 6250 3300 50  0001 C CNN
-F 3 "~" H 6250 3300 50  0001 C CNN
-	1    6250 3300
-	-1   0    0    1
+P 5300 3300
+F 0 "RV1" H 5231 3346 50  0000 R CNN
+F 1 "R_POT" H 5231 3255 50  0000 R CNN
+F 2 "Potentiometer_THT:Potentiometer_Vishay_T73YP_Vertical" H 5300 3300 50  0001 C CNN
+F 3 "~" H 5300 3300 50  0001 C CNN
+	1    5300 3300
+	1    0    0    1
 $EndComp
 $Comp
 L power:GND #PWR0112
 U 1 1 5F4900ED
-P 6250 3600
-F 0 "#PWR0112" H 6250 3350 50  0001 C CNN
-F 1 "GND" H 6255 3427 50  0000 C CNN
-F 2 "" H 6250 3600 50  0001 C CNN
-F 3 "" H 6250 3600 50  0001 C CNN
-	1    6250 3600
-	1    0    0    -1
+P 5300 3600
+F 0 "#PWR0112" H 5300 3350 50  0001 C CNN
+F 1 "GND" H 5305 3427 50  0000 C CNN
+F 2 "" H 5300 3600 50  0001 C CNN
+F 3 "" H 5300 3600 50  0001 C CNN
+	1    5300 3600
+	-1   0    0    -1
 $EndComp
 $Comp
@@
 	0    -1   -1   0
 $EndComp
-Wire Wire Line
-	6500 2850 6250 2850
-Connection ~ 6250 2850
 $Comp
 L MK_MCU:STM32L412K8Tx U2
@@
 L power:GND #PWR0122
 U 1 1 5F4859A8
-P 1700 1400
-F 0 "#PWR0122" H 1700 1150 50  0001 C CNN
-F 1 "GND" H 1705 1227 50  0000 C CNN
-F 2 "" H 1700 1400 50  0001 C CNN
-F 3 "" H 1700 1400 50  0001 C CNN
-	1    1700 1400
+P 1700 1550
+F 0 "#PWR0122" H 1700 1300 50  0001 C CNN
+F 1 "GND" H 1705 1377 50  0000 C CNN
+F 2 "" H 1700 1550 50  0001 C CNN
+F 3 "" H 1700 1550 50  0001 C CNN
+	1    1700 1550
 	1    0    0    -1
 $EndComp
@@
 	1700 1300 1600 1300
 Wire Wire Line
-	1700 1300 1700 1400
-Wire Wire Line
-	1700 1050 1700 1200
+	1700 1300 1700 1500
+Wire Wire Line
+	1700 950  1700 1000
 $Comp
 L Device:C C5
@@
 	3800 2250 3800 3150
 Wire Wire Line
-	6250 2850 6250 3150
-Wire Wire Line
-	6100 3300 5500 3300
-Wire Wire Line
 	5500 2950 5500 3300
 Wire Wire Line
-	6250 3600 6250 3450
+	5300 3600 5300 3450
 Wire Wire Line
 	4550 6050 4000 6050
@@
 NoConn ~ 3000 5850
 NoConn ~ 3000 6250
-NoConn ~ 4000 6550
-NoConn ~ 4000 6650
 NoConn ~ 4000 5450
 NoConn ~ 4000 5350
@@
 L power:+6V #PWR0103
 U 1 1 5F4FAFC7
-P 1700 1050
-F 0 "#PWR0103" H 1700 900 50  0001 C CNN
-F 1 "+6V" H 1715 1223 50  0000 C CNN
-F 2 "" H 1700 1050 50  0001 C CNN
-F 3 "" H 1700 1050 50  0001 C CNN
-	1    1700 1050
+P 1700 950
+F 0 "#PWR0103" H 1700 800 50  0001 C CNN
+F 1 "+6V" H 1715 1123 50  0000 C CNN
+F 2 "" H 1700 950 50  0001 C CNN
+F 3 "" H 1700 950 50  0001 C CNN
+	1    1700 950
 	1    0    0    -1
 $EndComp
@@
 Wire Wire Line
 	1750 3350 1750 3700
+$Comp
+L Device:Battery BT1
+U 1 1 5F4E7C7D
+P 1950 1250
+F 0 "BT1" H 2058 1296 50  0000 L CNN
+F 1 "Battery" H 2058 1205 50  0000 L CNN
+F 2 "MK_Footprints:BatteryHolder_Keystone_2477_4xAA" V 1950 1310 50  0001 C CNN
+F 3 "~" V 1950 1310 50  0001 C CNN
+	1    1950 1250
+	1    0    0    -1
+$EndComp
+Wire Wire Line
+	1950 1050 1950 1000
+Wire Wire Line
+	1950 1000 1700 1000
+Connection ~ 1700 1000
+Wire Wire Line
+	1700 1000 1700 1200
+Wire Wire Line
+	1950 1450 1950 1500
+Wire Wire Line
+	1950 1500 1700 1500
+Connection ~ 1700 1500
+Wire Wire Line
+	1700 1500 1700 1550
+Text GLabel 5950 4950 2    50   BiDi ~ 0
+SWDIO
+Text GLabel 5950 4850 2    50   Output ~ 0
+SWCLK
+$Comp
+L power:+3.3V #PWR0106
+U 1 1 5F56D562
+P 5950 4650
+F 0 "#PWR0106" H 5950 4500 50  0001 C CNN
+F 1 "+3.3V" H 5965 4823 50  0000 C CNN
+F 2 "" H 5950 4650 50  0001 C CNN
+F 3 "" H 5950 4650 50  0001 C CNN
+	1    5950 4650
+	1    0    0    -1
+$EndComp
+Wire Wire Line
+	5950 4650 5950 4750
+Wire Wire Line
+	5850 4750 5950 4750
+$Comp
+L power:GND #PWR0115
+U 1 1 5F5818FE
+P 5950 5150
+F 0 "#PWR0115" H 5950 4900 50  0001 C CNN
+F 1 "GND" H 5955 4977 50  0000 C CNN
+F 2 "" H 5950 5150 50  0001 C CNN
+F 3 "" H 5950 5150 50  0001 C CNN
+	1    5950 5150
+	1    0    0    -1
+$EndComp
+Wire Wire Line
+	5950 5050 5950 5150
+Wire Wire Line
+	5850 5050 5950 5050
+Text GLabel 4100 6550 2    50   BiDi ~ 0
+SWDIO
+Text GLabel 4100 6650 2    50   Output ~ 0
+SWCLK
+Wire Wire Line
+	4100 6550 4000 6550
+Wire Wire Line
+	4100 6650 4000 6650
+$Comp
+L Connector:Conn_01x04_Male J8
+U 1 1 5F607EBF
+P 5650 4850
+F 0 "J8" H 5758 5131 50  0000 C CNN
+F 1 "Conn_01x04_Male" H 5758 5040 50  0000 C CNN
+F 2 "Connector_PinHeader_2.54mm:PinHeader_1x04_P2.54mm_Vertical" H 5650 4850 50  0001 C CNN
+F 3 "~" H 5650 4850 50  0001 C CNN
+	1    5650 4850
+	1    0    0    -1
+$EndComp
+Wire Wire Line
+	5950 4950 5850 4950
+Wire Wire Line
+	5950 4850 5850 4850
+Wire Wire Line
+	6150 2850 6500 2850
+Wire Wire Line
+	5450 3300 5500 3300
+Wire Wire Line
+	5300 3050 5300 3150
+$Comp
+L power:+6V #PWR?
+U 1 1 5F6F4E43
+P 5300 3050
+F 0 "#PWR?" H 5300 2900 50  0001 C CNN
+F 1 "+6V" H 5315 3223 50  0000 C CNN
+F 2 "" H 5300 3050 50  0001 C CNN
+F 3 "" H 5300 3050 50  0001 C CNN
+	1    5300 3050
+	1    0    0    -1
+$EndComp
 $EndSCHEMATC
